Commit message: Package rl base navigation docker for Stretch3

File: src/goal_seeker_rl/urdf/turtlebot3_waffle_minimal.urdf (robot description, URDF)
Before this commit: robot turtlebot3_waffle_minimal, 3 links, 2 joints
Links:
- removed link base_scan
- added link camera_depth_frame
- added link camera_depth_optical_frame
- added link camera_link; visual box size=0.09 0.025 0.025
Joints:
- removed joint base_link_to_base_scan
- added joint base_link_to_camera_link: type fixed, parent base_link, child camera_link, origin xyz=0.069 -0.047 0.18 rpy=0 0 0
- added joint camera_depth_to_optical_frame: type fixed, parent camera_depth_frame, child camera_depth_optical_frame, origin xyz=0 0 0 rpy=-1.57079632679 0 -1.57079632679
- added joint camera_link_to_depth_frame: type fixed, parent camera_link, child camera_depth_frame, origin xyz=0 0 0 rpy=0 0 0
